Commit message: updated laser sensor

File: urdf/pocker_bot.xacro (robot description, xacro)
@@ -4,8 +4,10 @@
  <xacro:include filename="$(find pocker_bot_description)/urdf/materials.xacro" />
  <xacro:include filename="$(find pocker_bot_description)/urdf/wheel_macros.xacro" />
+  <xacro:include filename="$(find pocker_bot_vrep_description)/urdf/sensor_macros.xacro" />
 <!-- Namespaces of links -->
   <xacro:property name="base_name" value="base_link" />
   <xacro:property name="left_wheel" value="left_wheel_link" />
   <xacro:property name="right_wheel" value="right_wheel_link" />
+  <xacro:property name="laser_sensor" value="laser_sensor" />
 <!-- Configuration of the base of the robot-->
  <xacro:property name="bot_height" value="0.054024" />
@@ -16,4 +18,7 @@
  <xacro:property name="wheel_radius" value="${(bot_height/2)+(caster_radius)}" />
  <xacro:property name="wheel_thickness" value="0.012" />
+   <!-- Configuration of sensor -->
+ <xacro:property name="sensor_thickness" value="0.035" />
+ <xacro:property name="sensor_radius" value="0.025" />
  	<link name="${base_name}">
     <inertial>
@@ -91,3 +96,5 @@
   <xacro:link_wheel name="${right_wheel}" thickness="${wheel_thickness}" radius="${wheel_radius}" origin_xyz="0 0 0" mesh_filename="wheel.dae" visual_origin_rpy="0 0 -1.57"/>
   <xacro:joint_wheel name="joint_${right_wheel}" parent="${base_name}" child="${right_wheel}" origin_xyz="0 ${-bot_base_radius-0.013} ${(bot_height/2)+caster_radius}" />
+    <xacro:sensor name="${laser_sensor}" thickness="${sensor_thickness}" radius="${sensor_radius}" origin_xyz="0 0 ${-sensor_thickness/2}" mesh_filename="hokuyo.dae" visual_origin_rpy=" 0 0 ${-sensor_thickness/2}"/>
+  <xacro:sensor_joint name="sensor_joint_${laser_sensor}" parent="${base_name}" child="${laser_sensor}" origin_xyz="${(3/4)*bot_base_radius} 0 ${bot_height+caster_radius+(sensor_thickness)}" />
 </robot>
